Commit message: Add robot wheels and wheel joints

File: ros2_ws/src/simple_robot_description/urdf/robot.urdf (robot description, URDF)
Before this commit: robot simple_robot, 1 links, 0 joints
Links:
- added link left_wheel; visual cylinder length=0.02 radius=0.05
- added link right_wheel; visual cylinder length=0.02 radius=0.05
Joints:
- added joint left_wheel_joint: type continuous, parent base_link, child left_wheel, origin xyz=0 0.15 -0.05, axis 0 1 0
- added joint right_wheel_joint: type continuous, parent base_link, child right_wheel, origin xyz=0 -0.15 -0.05, axis 0 1 0

Commit message: Add caster wheel

File: ros2_ws/src/simple_robot_description/urdf/robot.urdf (robot description, URDF)
Before this commit: robot simple_robot, 3 links, 2 joints
Links:
- added link caster_wheel; visual sphere radius=0.035
Joints:
- added joint caster_joint: type fixed, parent base_link, child caster_wheel, origin xyz=-0.18 0 -0.06

Commit message: Add camera link to robot URDF

File: ros2_ws/src/simple_robot_description/urdf/robot.urdf (robot description, URDF)
Before this commit: robot simple_robot, 4 links, 3 joints
Links:
- added link camera_link; visual box size=0.05 0.05 0.05
Joints:
- added joint camera_joint: type fixed, parent base_link, child camera_link, origin xyz=0.25 0 0.08

Commit message: Add RViz configuration

File: ros2_ws/src/simple_robot_description/urdf/robot.urdf (robot description, URDF)
Before this commit: robot simple_robot, 5 links, 4 joints
Links:
- added link lidar_link; visual cylinder length=0.03 radius=0.04
Joints:
- added joint lidar_joint: type fixed, parent base_link, child lidar_link, origin xyz=0.1 0 0.1
